File: schematics/KICAD/RE-Mellanox connectX-3PRO Lenovo ML adapter - 00FP652/RE-Mellanox connectX-3PRO Lenovo ML adapter - 00FP652.kicad_sch (KiCad schematic)
At the start: 0 parts

Commit message: Update KiCad schematic and project metadata
Populate and update KiCad project files for the RE-Mellanox connectX-3PRO Lenovo ML adapter: expanded .kicad_sch with symbol definitions and schematic content, updated .kicad_pro with design rules, ERC, BOM and drawing settings, and adjusted net inspector preferences in .kicad_prl. Added backup ZIP files and fp-info-cache for the project.
Parts:
- added J1, J2: 1704320001, my_stuff:AMT0440005DB0000G, symbol qsfp:1704320001
- added U1: SN74CB3Q3253DBQR, DBQ16, symbol SN74CB3Q3253:SN74CB3Q3253DBQR
